Commit message: Running the second launchfile spawns something in Gazebo but alas. It is just a grey ball.

File: src/bb8/urdf/bb8_dummy.xacro (robot description, xacro)
@@ -26,5 +26,5 @@
               <origin rpy="0 0 0" xyz="0 0.0 ${-1*r}" />
               <geometry>
-                <mesh filename="package://bb_8_description/meshes/bb8/ball_bb8/ball.dae" scale="1 1 1"/>
+                <mesh filename="package://bb8/src/meshes/ball.dae" scale="1 1 1"/>
               </geometry>
             </visual>

File: src/bb8/urdf/bb8_head.xacro (robot description, xacro)
@@ -17,5 +17,5 @@
               <origin rpy="0 0 3.14" xyz="0 0.0 -${sphere_radius}" />
               <geometry>
-                <mesh filename="package://bb_8_description/meshes/bb8/head_bb8/head.dae" scale="1 1 1"/>
+                <mesh filename="package://bb8/src/meshes/head.dae" scale="1 1 1"/>
               </geometry>
             </visual>
