Commit message: spawn_bb8_launch runs and starts /cmd_vel but no visual elements, spawn_bb8_2_launch runs and spawns visual elements but no /cmd_vel

File: src/bb8/urdf/bb8_head.xacro (robot description, xacro)
@@ -6,5 +6,5 @@
               <origin rpy="0 0 0" xyz="0.0 0.0 0.0" />
               <mass value="${head_mass}" />
-              <sphere_inertia mass="${head_mass}" r="${head_radius}" />
+              <sphere_inertia mass="${head_mass}" r="${head_radius}"/>
             </inertial>
             <collision>

File: src/bb8/urdf2/bb8.gazebo.xacro (robot description, xacro)
@@ -10,4 +10,11 @@
     <maxVel>10.0</maxVel>
     <minDepth>0.0005</minDepth>
+    <visual>
+      <geometry>
+        <!-- Assuming you have a geometry set for the base_link, such as a cylinder -->
+        <cylinder radius="0.2" length="0.5"/>
+      </geometry>
+      <material>Gazebo/Orange</material>
+    </visual>
   </gazebo>
   <gazebo reference="base_rotation_link">
@@ -56,4 +63,18 @@
     <maxVel>1.0</maxVel>
     <minDepth>0.003</minDepth>
+    <visual>
+      <geometry>
+        <mesh>
+          <uri>model://bb8/meshes/head_bb8.dae"</uri>
+        </mesh>
+      </geometry>
+    </visual>
+    <collision>
+      <geometry>
+        <mesh>
+          <uri>model://bb8/meshes/head_bb8.dae"</uri>
+        </mesh>
+      </geometry>
+    </collision>
   </gazebo>
   <!-- gazebo reference="wheel_joint">

File: src/bb8/urdf2/bb8.urdf (robot description, URDF)
Before this commit: robot bb_8, 5 links, 4 joints
Links:
- link head_link: geometry collision sphere radius=0.2; visual sphere radius=0.2
