Commit message: working on getting test_command.py to work (does not rn). rn if you run "ros2 launch gazebo_ros gazebo.launch.py" in one terminal, run "ros2 launch bb8 spawn_bb8_launch.py" in the second terminal, and then run "ros2 topic pub /cmd_vel geometry_msgs/msg/Twist "{linear: {x: 0.5, y: 0.0, z: 0.0}, angular: {x: 0.0, y: 0.0, z: 0.5}}"" in the third terminal you can move him. he is still grey ball.

File: src/bb8/urdf/bb8.xacro (robot description, xacro)
@@ -13,5 +13,8 @@
       <mass value="${robot_mass}"/>
       <origin rpy="0 0 0" xyz="0 0 0"/>
-      <box_inertia mass="${robot_mass}" x="${sphere_radius*2.0}" y="${sphere_radius*2.0}" z="${sphere_radius*2.0}" />
+      <!--box_inertia mass="${robot_mass}" x="${sphere_radius*2.0}" y="${sphere_radius*2.0}" z="${sphere_radius*2.0}" -->
+      <inertia ixx="0.01" ixy="0.0" ixz="0.0"
+             iyy="0.01" iyz="0.0"
+             izz="0.01" /> <!--replace later w calculated vals-->
     </inertial>
     <!-- body -->

File: src/bb8/urdf/bb8_dummy.xacro (robot description, xacro)
@@ -15,5 +15,8 @@
               <mass value="0.2"/>
               <origin rpy="0 1.5707 1.5707" xyz="0 0 0"/>
-               <cylinder_inertia mass="0.2" r="${r}" l="${l}" />
+              <!--cylinder_inertia mass="0.2" r="${r}" l="${l}" -->
+              <inertia ixx="0.01" ixy="0.0" ixz="0.0"
+             iyy="0.01" iyz="0.0"
+             izz="0.01" /> <!--replace later w calculated vals-->
             </inertial>
             <collision name="link_right_wheel_collision">

File: src/bb8/urdf/bb8_head.xacro (robot description, xacro)
@@ -6,5 +6,8 @@
               <origin rpy="0 0 0" xyz="0.0 0.0 0.0" />
               <mass value="${head_mass}" />
-              <sphere_inertia mass="${head_mass}" r="${head_radius}"/>
+              <!--sphere_inertia mass="${head_mass}" r="${head_radius}"-->
+              <inertia ixx="0.01" ixy="0.0" ixz="0.0"
+             iyy="0.01" iyz="0.0"
+             izz="0.01" /> <!--replace later w calculated vals-->
             </inertial>
             <collision>
@@ -15,7 +18,9 @@
             </collision>
             <visual>
-              <origin rpy="0 0 3.14" xyz="0 0.0 -${sphere_radius}" />
+              <!--origin rpy="0 0 3.14" xyz="0 0.0 -${sphere_radius}" -->
               <geometry>
-                <mesh filename="package://bb8/src/meshes/head.dae" scale="1 1 1"/>
+                <!--mesh filename="package://bb8/src/meshes/head.dae" scale="1 1 1"-->
+                <!--mesh filename="file://bb8/src/meshes/head.dae" -->
+                <sphere radius="${sphere_radius}"/>
               </geometry>
             </visual>

File: src/bb8/urdf/macros.xacro (robot description, xacro)
@@ -18,13 +18,13 @@
       </xacro:macro>
     <xacro:macro name="sphere_inertia" params="mass r">
-    <inertia
-          ixx="${2*mass*r*r/5}"
-    			ixy = "0"
-    			ixz = "0"
-    			iyy="${2*mass*r*r/5}"
-    			iyz = "0"
-    			izz="${2*mass*r*r/5}"
-    />
-  </xacro:macro>
+      <inertia
+            ixx="${2*mass*r*r/5}"
+            ixy = "0"
+            ixz = "0"
+            iyy="${2*mass*r*r/5}"
+            iyz = "0"
+            izz="${2*mass*r*r/5}"
+      />
+    </xacro:macro>
     <xacro:macro  name="link_wheel" params="name r l incr">
         <link name="${name}">
@@ -32,5 +32,8 @@
               <mass value="0.2"/>
               <origin rpy="0 1.5707 1.5707" xyz="0 0 0"/>
-               <cylinder_inertia mass="0.2" r="${r}" l="${l}" />
+               <!--cylinder_inertia mass="0.2" r="${r}" l="${l}" -->
+              <inertia ixx="0.01" ixy="0.0" ixz="0.0"
+             iyy="0.01" iyz="0.0"
+             izz="0.01" /> <!--replace later w calculated vals-->
             </inertial>
             <collision name="link_right_wheel_collision">

Commit message: bb8 rendering and running test files in scripts folder with spawn_bb8_launch.py

File: src/bb8/urdf/bb8.xacro (robot description, xacro)
@@ -24,4 +24,12 @@
       </geometry>
     </collision>
+    <visual>
+      <origin rpy="0 0 0" xyz="0 0.0 ${sphere_radius}" />
+      <geometry>
+        <sphere radius="${sphere_radius}"/>
+        <!--mesh filename="package://bb8/src/meshes/ball.dae" scale="1 1 1"/-->
+      </geometry>
+      <material name="Gazebo/Orange"/>
+    </visual>
   </link>
   <xacro:link_wheel name="link_right_wheel" r="${sphere_radius}" l="${wheel_thickness}" incr="${wheel_increment}"/>
@@ -30,4 +38,4 @@
   <xacro:joint_wheel name="joint_left_wheel" child="link_left_wheel" origin_xyz="0 ${-1*sphere_radius/2.0} 0" />
   <xacro:bb_8_dummy  name="bb_8_dummy" parent="link_chassis" r="${sphere_radius}" l="${wheel_thickness}" incr="${wheel_increment}"/>
-  <xacro:bb_8_head  parent="link_chassis"/>
+  <xacro:bb_8_head parent="link_chassis"/>
 </robot>

File: src/bb8/urdf/bb8_dummy.xacro (robot description, xacro)
@@ -26,10 +26,4 @@
               </geometry>
             </collision>
-            <visual>
-              <origin rpy="0 0 0" xyz="0 0.0 ${-1*r}" />
-              <geometry>
-                <mesh filename="package://bb8/src/meshes/ball.dae" scale="1 1 1"/>
-              </geometry>
-            </visual>
           </link>
           <joint name="direction_joint" type="continuous">

File: src/bb8/urdf/bb8_head.xacro (robot description, xacro)
@@ -4,5 +4,5 @@
         <link name="head_link">
             <inertial>
-              <origin rpy="0 0 0" xyz="0.0 0.0 0.0" />
+              <origin rpy="0 0 0" xyz="0.0 0.0 ${sphere_radius}" />
               <mass value="${head_mass}" />
               <!--sphere_inertia mass="${head_mass}" r="${head_radius}"-->
@@ -12,5 +12,5 @@
             </inertial>
             <collision>
-              <origin rpy="0 0 0" xyz="0 0 ${sphere_radius}" />
+              <origin rpy="0 0 0" xyz="0 0 ${head_radius}" />
               <geometry>
                 <sphere radius="${head_radius}"/>
@@ -18,9 +18,9 @@
             </collision>
             <visual>
-              <!--origin rpy="0 0 3.14" xyz="0 0.0 -${sphere_radius}" -->
+              <origin rpy="0 0 3.14" xyz="0 0.0 ${2*sphere_radius}" />
               <geometry>
                 <!--mesh filename="package://bb8/src/meshes/head.dae" scale="1 1 1"-->
                 <!--mesh filename="file://bb8/src/meshes/head.dae" -->
-                <sphere radius="${sphere_radius}"/>
+                <sphere radius="${head_radius}"/>
               </geometry>
             </visual>

File: src/bb8/urdf/macros.xacro (robot description, xacro)
@@ -43,4 +43,12 @@
               </geometry>
             </collision>
+            <visual name="${name}_visual">
+                <origin rpy="0 1.5707 1.5707" xyz="0 0 0"/>
+                <geometry>
+                    <cylinder length="${l}" radius="${r + incr}"/>
+                </geometry>
+                <!-- Define the material for the wheel. You can customize this -->
+                <material name="Gazebo/Blue"/>
+            </visual>
         </link>
     </xacro:macro >

Commit message: meshes showing up

File: src/bb8/urdf/bb8.xacro (robot description, xacro)
@@ -27,14 +27,14 @@
       <origin rpy="0 0 0" xyz="0 0.0 ${sphere_radius}" />
       <geometry>
-        <sphere radius="${sphere_radius}"/>
-        <!--mesh filename="package://bb8/src/meshes/ball.dae" scale="1 1 1"/-->
+        <!--sphere radius="${sphere_radius}"/-->
+        <mesh filename="package://bb8/meshes/ball.dae" scale="1 1 1"/>
       </geometry>
-      <material name="Gazebo/Orange"/>
+      <!--material name="Gazebo/Orange"/-->
     </visual>
   </link>
   <xacro:link_wheel name="link_right_wheel" r="${sphere_radius}" l="${wheel_thickness}" incr="${wheel_increment}"/>
-  <xacro:joint_wheel name="joint_right_wheel" child="link_right_wheel" origin_xyz="0 ${sphere_radius/2.0} 0" />
+  <xacro:joint_wheel name="joint_right_wheel" child="link_right_wheel" origin_xyz="0 ${sphere_radius/2} 0" />
   <xacro:link_wheel name="link_left_wheel" r="${sphere_radius}" l="${wheel_thickness}" incr="${wheel_increment}"/>
-  <xacro:joint_wheel name="joint_left_wheel" child="link_left_wheel" origin_xyz="0 ${-1*sphere_radius/2.0} 0" />
+  <xacro:joint_wheel name="joint_left_wheel" child="link_left_wheel" origin_xyz="0 ${-1*sphere_radius/2} 0" />
   <xacro:bb_8_dummy  name="bb_8_dummy" parent="link_chassis" r="${sphere_radius}" l="${wheel_thickness}" incr="${wheel_increment}"/>
   <xacro:bb_8_head parent="link_chassis"/>

File: src/bb8/urdf/bb8_dummy.xacro (robot description, xacro)
@@ -32,5 +32,5 @@
             <child link="${name}_base_direction_link" />
             <axis xyz="0 1 0" />
-            <limit effort="1000.0" velocity="100.0" />
+            <limit effort="1000.0" velocity="1000.0" />
           </joint>
         <transmission name="direction_joint_trans">

File: src/bb8/urdf/bb8_head.xacro (robot description, xacro)
@@ -4,5 +4,6 @@
         <link name="head_link">
             <inertial>
-              <origin rpy="0 0 0" xyz="0.0 0.0 ${sphere_radius}" />
+              <!--origin rpy="0 0 0" xyz="0.0 0.0 ${sphere_radius}" /-->
+              <origin rpy="0 0 0" xyz="0.0 0.0 0.0" />
               <mass value="${head_mass}" />
               <!--sphere_inertia mass="${head_mass}" r="${head_radius}"-->
@@ -12,5 +13,6 @@
             </inertial>
             <collision>
-              <origin rpy="0 0 0" xyz="0 0 ${head_radius}" />
+              <!--origin rpy="0 0 0" xyz="0 0 ${head_radius}" /-->
+              <origin rpy="0 0 0" xyz="0 0 ${sphere_radius}" />
               <geometry>
                 <sphere radius="${head_radius}"/>
@@ -18,9 +20,8 @@
             </collision>
             <visual>
-              <origin rpy="0 0 3.14" xyz="0 0.0 ${2*sphere_radius}" />
+              <origin rpy="0 0 3.14" xyz="0 0.0 ${sphere_radius}" />
               <geometry>
-                <!--mesh filename="package://bb8/src/meshes/head.dae" scale="1 1 1"-->
-                <!--mesh filename="file://bb8/src/meshes/head.dae" -->
-                <sphere radius="${head_radius}"/>
+                <mesh filename="package://bb8/meshes/head.dae" scale="1 1 1"/>
+                <!--sphere radius="${head_radius}"/-->
               </geometry>
             </visual>
@@ -31,5 +32,5 @@
             <child link="head_link" />
             <axis xyz="0 0 1" />
-            <limit effort="1.0" velocity="1.0" lower="-1e+16" upper="1e+16"/>
+            <limit effort="1000.0" velocity="1000.0" lower="-1e+16" upper="1e+16"/>
           </joint>
         <transmission name="head_joint_trans">

Commit message: bb8 FINALLY showing mesh and correct proportions, updated wheel radius to .55

File: src/bb8/urdf/bb8.xacro (robot description, xacro)
@@ -21,9 +21,10 @@
     <collision name="collision_chassis">
       <geometry>
-        <box size="${sphere_radius*2.0} ${sphere_radius*2.0} ${sphere_radius*2.0}"/>
+        <box size="${sphere_radius} ${sphere_radius} ${sphere_radius}"/>
       </geometry>
     </collision>
     <visual>
-      <origin rpy="0 0 0" xyz="0 0.0 ${sphere_radius}" />
+      <!--origin rpy="0 0 0" xyz="0 0.0 ${sphere_radius}" /-->
+      <origin rpy="0 0 0" xyz="0 0.0 -${sphere_radius}" />
       <geometry>
         <!--sphere radius="${sphere_radius}"/-->
@@ -33,8 +34,8 @@
     </visual>
   </link>
-  <xacro:link_wheel name="link_right_wheel" r="${sphere_radius}" l="${wheel_thickness}" incr="${wheel_increment}"/>
-  <xacro:joint_wheel name="joint_right_wheel" child="link_right_wheel" origin_xyz="0 ${sphere_radius/2} 0" />
-  <xacro:link_wheel name="link_left_wheel" r="${sphere_radius}" l="${wheel_thickness}" incr="${wheel_increment}"/>
-  <xacro:joint_wheel name="joint_left_wheel" child="link_left_wheel" origin_xyz="0 ${-1*sphere_radius/2} 0" />
+  <xacro:link_wheel name="link_right_wheel" r="${sphere_radius+.2}" l="${wheel_thickness}" incr="${wheel_increment}"/>
+  <xacro:joint_wheel name="joint_right_wheel" child="link_right_wheel" origin_xyz="0 ${sphere_radius} 0" />
+  <xacro:link_wheel name="link_left_wheel" r="${sphere_radius+.2}" l="${wheel_thickness}" incr="${wheel_increment}"/>
+  <xacro:joint_wheel name="joint_left_wheel" child="link_left_wheel" origin_xyz="0 ${-1*sphere_radius} 0" />
   <xacro:bb_8_dummy  name="bb_8_dummy" parent="link_chassis" r="${sphere_radius}" l="${wheel_thickness}" incr="${wheel_increment}"/>
   <xacro:bb_8_head parent="link_chassis"/>

File: src/bb8/urdf/bb8_head.xacro (robot description, xacro)
@@ -14,5 +14,5 @@
             <collision>
               <!--origin rpy="0 0 0" xyz="0 0 ${head_radius}" /-->
-              <origin rpy="0 0 0" xyz="0 0 ${sphere_radius}" />
+              <origin rpy="0 0 0" xyz="0 0 -${sphere_radius}" />
               <geometry>
                 <sphere radius="${head_radius}"/>
@@ -20,5 +20,6 @@
             </collision>
             <visual>
-              <origin rpy="0 0 3.14" xyz="0 0.0 ${sphere_radius}" />
+              <!--origin rpy="0 0 3.14" xyz="0 0.0 ${sphere_radius}" /-->
+              <origin rpy="0 0 3.14" xyz="0 0.0 -${sphere_radius}" />
               <geometry>
                 <mesh filename="package://bb8/meshes/head.dae" scale="1 1 1"/>

Commit message: bb8 looks great and is shmoovin

File: src/bb8/urdf/bb8.xacro (robot description, xacro)
@@ -25,5 +25,6 @@
     </collision>
     <visual>
-      <origin rpy="0 0 0" xyz="0 0.0 ${sphere_radius}" />
+      <!--origin rpy="0 0 0" xyz="0 0.0 ${sphere_radius}" /-->
+      <origin rpy="0 0 0" xyz="0 0.0 ${-1*sphere_radius}" />
       <geometry>
         <!--sphere radius="${sphere_radius}"/-->

File: src/bb8/urdf/bb8_head.xacro (robot description, xacro)
@@ -14,5 +14,6 @@
             <collision>
               <!--origin rpy="0 0 0" xyz="0 0 ${head_radius}" /-->
-              <origin rpy="0 0 0" xyz="0 0 ${sphere_radius}" />
+              <!--origin rpy="0 0 0" xyz="0 0 ${sphere_radius}" /-->
+              <origin rpy="0 0 0" xyz="0 0 0" />
               <geometry>
                 <sphere radius="${head_radius}"/>
@@ -20,5 +21,6 @@
             </collision>
             <visual>
-              <origin rpy="0 0 3.14" xyz="0 0.0 ${sphere_radius}" />
+              <!--origin rpy="0 0 3.14" xyz="0 0.0 ${sphere_radius}" /-->
+              <origin rpy="0 0 3.14" xyz="0 0.0 -${sphere_radius}" />
               <geometry>
                 <mesh filename="package://bb8/meshes/head.dae" scale="1 1 1"/>
